Commit message: Tried to add car to rviz, failed, cried, and now i wanna kill myself

File: ros2_ackermann_gazebo/urdf/test_ackermann_drive.xacro.urdf (robot description, URDF)
Before this commit: robot ackermann_drive, 10 links, 9 joints
Links:
- link camera_link: geometry collision box size=0.01 0.01 0.01; visual box size=0.01 0.01 0.01
- link chassis: geometry collision box size=0.6 0.3 0.05; visual box size=0.6 0.3 0.05
- link front_left_wheel: geometry collision cylinder length=0.04 radius=0.05; visual cylinder length=0.04 radius=0.05
- link front_right_wheel: geometry collision cylinder length=0.04 radius=0.05; visual cylinder length=0.04 radius=0.05
- link rear_left_wheel: geometry collision cylinder length=0.04 radius=0.05; visual cylinder length=0.04 radius=0.05
- link rear_right_wheel: geometry collision cylinder length=0.04 radius=0.05; visual cylinder length=0.04 radius=0.05
Joints:
- joint camera_joint: origin xyz=1 0 1 rpy=0 0 0 -> xyz=0 0 0.23 rpy=0 0 0
- joint chassis_joint: origin xyz=0.8 0 0.5 rpy=0 0 0 -> xyz=-0.08 0 0.055 rpy=0 0 0
- joint left_wheel_steering_joint: origin xyz=0.9 -0.5 -0.2 rpy=1.57 0 0 -> xyz=0.18 -0.1301 -0.005 rpy=1.57 0 0
- joint rear_left_wheel_joint: origin xyz=-0.8 0.5 -0.2 rpy=-1.57 0 0 -> xyz=-0.18 0.1301 -0.005 rpy=-1.57 0 0
- joint rear_right_wheel_joint: origin xyz=-0.8 -0.5 -0.2 rpy=-1.57 0 0 -> xyz=-0.18 -0.1301 -0.005 rpy=-1.57 0 0
- joint right_wheel_steering_joint: origin xyz=0.9 0.5 -0.2 rpy=1.57 0 0 -> xyz=0.18 0.1301 -0.005 rpy=1.57 0 0

Commit message: [RAR-58] Better simulation

File: ros2_ackermann_gazebo/urdf/test_ackermann_drive.xacro.urdf (robot description, URDF)
Before this commit: robot ackermann_drive, 10 links, 9 joints
Joints:
- joint camera_optical_joint: origin xyz=0 0 0 rpy=-1.5707963267948966 0 -1.5707963267948966 -> xyz=-0.000029859 0.00012 0 rpy=-1.5707963267948966 0 -1.5707963267948966

Commit message: [RAR-42-ImageController] Add: run_through_script.py allowing to change the car's possition Add: working function for path creation Add: shutdown function for the node Change: setup image_logic for interaction with the nav2 controll stack

File: ros2_ackermann_gazebo/urdf/test_ackermann_drive.xacro.urdf (robot description, URDF)
Before this commit: robot ackermann_drive, 10 links, 9 joints
Links:
- link chassis: geometry collision box size=0.6 0.3 0.04; visual box size=0.6 0.3 0.02
Joints:
- joint chassis_joint: origin xyz=-0.08 0 0.055 rpy=0 0 0 -> xyz=-0.08 0 0.05 rpy=0 0 0
- joint left_wheel_steering_joint: origin xyz=0.18 -0.1301 -0.005 rpy=1.57 0 0 -> xyz=0.18 -0.1301 -0.00 rpy=1.57 0 0
- joint rear_left_wheel_joint: origin xyz=-0.18 0.1301 -0.005 rpy=-1.57 0 0 -> xyz=-0.18 0.1301 -0.00 rpy=-1.57 0 0
- joint rear_right_wheel_joint: origin xyz=-0.18 -0.1301 -0.005 rpy=-1.57 0 0 -> xyz=-0.18 -0.1301 -0.00 rpy=-1.57 0 0
- joint right_wheel_steering_joint: origin xyz=0.18 0.1301 -0.005 rpy=1.57 0 0 -> xyz=0.18 0.1301 -0.00 rpy=1.57 0 0

Commit message: kinda works, slow reactiveness and small problems with computervision.

File: ros2_ackermann_gazebo/urdf/test_ackermann_drive.xacro.urdf (robot description, URDF)
Before this commit: robot ackermann_drive, 10 links, 9 joints
Links:
- link chassis: geometry collision box size=0.6 0.3 0.04; visual box size=0.5 0.3 0.002

Commit message: add ros2_ackermann_gazebo

File: ros2_ackermann_gazebo/urdf/test_ackermann_drive.xacro.urdf (robot description, URDF)
Before this commit: robot ackermann_drive, 10 links, 9 joints
Links:
- link camera_link: geometry collision box size=0.01 0.01 0.01; visual box size=0.01 0.01 0.01
- link chassis: geometry collision box size=0.6 0.3 0.04; visual box size=0.5 0.3 0.002
- link front_left_wheel: geometry collision cylinder length=0.04 radius=0.05; visual cylinder length=0.04 radius=0.05
- link front_right_wheel: geometry collision cylinder length=0.04 radius=0.05; visual cylinder length=0.04 radius=0.05
- link rear_left_wheel: geometry collision cylinder length=0.04 radius=0.05; visual cylinder length=0.04 radius=0.05
- link rear_right_wheel: geometry collision cylinder length=0.04 radius=0.05; visual cylinder length=0.04 radius=0.05
Joints:
- joint camera_joint: origin xyz=1 0 1 rpy=0 0 0 -> xyz=0 0 0.23 rpy=0 0 0
- joint camera_optical_joint: origin xyz=0 0 0 rpy=-1.5707963267948966 0 -1.5707963267948966 -> xyz=-0.000029859 0.00012 0 rpy=-1.5707963267948966 0 -1.5707963267948966
- joint chassis_joint: origin xyz=0.8 0 0.5 rpy=0 0 0 -> xyz=-0.08 0 0.05 rpy=0 0 0
- joint left_wheel_steering_joint: origin xyz=0.9 -0.5 -0.2 rpy=1.57 0 0 -> xyz=0.18 -0.1301 -0.00 rpy=1.57 0 0
- joint rear_left_wheel_joint: origin xyz=-0.8 0.5 -0.2 rpy=-1.57 0 0 -> xyz=-0.18 0.1301 -0.00 rpy=-1.57 0 0
- joint rear_right_wheel_joint: origin xyz=-0.8 -0.5 -0.2 rpy=-1.57 0 0 -> xyz=-0.18 -0.1301 -0.00 rpy=-1.57 0 0
- joint right_wheel_steering_joint: origin xyz=0.9 0.5 -0.2 rpy=1.57 0 0 -> xyz=0.18 0.1301 -0.00 rpy=1.57 0 0
